Commit message: fix(krsbi_description): remove redundant pi definition in properties.xacro
- xacro already provides pi as built-in constant
- Fixes 'redefining global symbol: pi' warning
- Resolves launch failure due to stderr output

File: krsbi_description/urdf/properties.xacro (robot description, xacro)
@@ -9,5 +9,5 @@
 <robot xmlns:xacro="http://www.ros.org/wiki/xacro" name="properties">
   <!-- ==================== MATH CONSTANTS ==================== -->
-  <xacro:property name="pi" value="3.14159265359"/>
+  <!-- pi is already defined by xacro globally -->
   <xacro:property name="cos_60" value="0.5"/>
   <xacro:property name="sin_60" value="0.866025403784"/>
